Commit message: Update mowbot-T2.urdf.xacro

File: mowbot_description/urdf/mowbot-T2.urdf.xacro (robot description, xacro)
@@ -2,7 +2,7 @@
 <robot xmlns:xacro="http://www.ros.org/wiki/xacro" name="mowbot-T2">
   <xacro:property name="PI" value="3.1415926535897931"/>
-  <xacro:property name="length" value="1.34"/>
-  <xacro:property name="width" value="1.26"/>
-  <xacro:property name="height" value="0.662"/>
+  <xacro:property name="length" value="1.39"/>
+  <xacro:property name="width" value="1.40"/>
+  <xacro:property name="height" value="0.765"/>
   <material name="red">
     <color rgba="0.8 0.0 0.0 1.0"/>
@@ -32,5 +32,5 @@
     <parent link="base_footprint"/>
     <child link="base_link"/>
-    <origin xyz="0.0 0.0 0.335" rpy="0.0 0.0 0.0"/>
+    <origin xyz="0.0 0.0 0.2" rpy="0.0 0.0 0.0"/>
   </joint>
   <link name="imu_link">
@@ -45,5 +45,5 @@
     <parent link="base_link"/>
     <child link="imu_link"/>
-    <origin xyz="-0.14 0.0 ${height - 0.335 + 0.015}" rpy="0.0 0.0 0.0"/>
+    <origin xyz="-0.415 0.0 ${height - 0.2 + 0.015}" rpy="0.0 0.0 0.0"/>
     <!-- <origin xyz="-0.14 0.0 ${height - 0.335 + 0.015}" rpy="0.0 0.0 ${PI}"/> -->
   </joint>
@@ -65,5 +65,5 @@
     <parent link="base_link"/>
     <child link="laser_link"/>
-    <origin xyz="0.2 0.0 ${height - 0.335 + 0.2}" rpy="0.0 0.0 ${PI}"/>
+    <origin xyz="0.415 0.0 ${height - 0.2 + 0.2}" rpy="0.0 0.0 ${PI}"/>
   </joint>
   <link name="camera_link">
@@ -78,5 +78,5 @@
     <parent link="base_link"/>
     <child link="camera_link"/>
-    <origin xyz="0.55 0.0 ${height - 0.335 + 0.08}" rpy="0.0 0.0 0.0"/>
+    <origin xyz="0.55 0.0 ${height - 0.2 + 0.08}" rpy="0.0 0.0 0.0"/>
   </joint>
   <link name="uwb_tag_link">
@@ -92,5 +92,5 @@
     <parent link="base_link"/>
     <child link="gps_right_link"/>
-    <origin xyz="-0.1 -0.52 ${height - 0.335 -0.05}" rpy="0.0 0.0 0.0"/>
+    <origin xyz="-0.39 -0.355 ${height - 0.2 -0.05}" rpy="0.0 0.0 0.0"/>
   </joint>
   <link name="gps_left_link">
@@ -99,5 +99,5 @@
     <parent link="base_link"/>
     <child link="gps_left_link"/>
-    <origin xyz="-0.1 0.52 ${height - 0.335 - 0.05}" rpy="0.0 0.0 0.0"/>
+    <origin xyz="-0.39 0.355 ${height - 0.2 - 0.05}" rpy="0.0 0.0 0.0"/>
   </joint>
 </robot>

Commit message: Corrected the position of the laser joint in mowbot-T2.urdf.xacro by adjusting the x-coordinate from 0.415 to -0.415.

File: mowbot_description/urdf/mowbot-T2.urdf.xacro (robot description, xacro)
@@ -65,5 +65,5 @@
     <parent link="base_link"/>
     <child link="laser_link"/>
-    <origin xyz="0.415 0.0 ${height - 0.2 + 0.2}" rpy="0.0 0.0 ${PI}"/>
+    <origin xyz="-0.415 0.0 ${height - 0.2 + 0.2}" rpy="0.0 0.0 ${PI}"/>
   </joint>
   <link name="camera_link">
